File: pcb/diplomna_2024_sensors_pcb_layout/diplomna_2024_sensors_pcb_layout.kicad_pcb (KiCad board)
At the start: 4 copper layers, 95 x 95 mm, 12 parts

Commit message: PC UPDATES
Parts:
- added REF**: PinHeader_1x05_P2.54mm_Vertical, Connector_PinHeader_2.54mm:PinHeader_1x05_P2.54mm_Vertical, F.Cu at (174.3, 68.0)
Connections:
- J** pad 1: (no net) -> GND
- J** pad 116: (no net) -> SQW
- J** pad 2: (no net) -> GND
- J** pad 30: (no net) -> GND
- J** pad 31: (no net) -> GND
Routing:
- net SDA: track 85.0 -> 119.9 mm
- net SCL: track 91.4 -> 112.6 mm
- net SQW: track 0.00 -> 8.98 mm
- net VIN: track 304.0 -> 311.8 mm
Other:
- board text added: "RTC"
- board text added: "v1"
